File: PCB/v2/moth_v2.sch (EAGLE design)
At the start: 64 parts

Commit message: finished the v2 PCB
Parts:
- removed 3.3V, 5V, BAT+, GND, SCL, SCL0, SCL1, SDA, SDA0, SDA1: TEST_POINT_LARGE, nathans-custom-parts:TEST_POINT_LARGE
- removed B1: TEENSY-3.1NOSILK, SparkFun-Boards:TEENSY-3.1NOSILK
- removed BAT_IN: B2B-PH-K, con-jst-ph:B2B-PH-K
- removed NC11, NC12: 0.1uf, SparkFun-Capacitors:5.6PF-0603-50V-5%
- removed NEO_01, NEO_02, NEO_03, NEO_04, NEO_05, NEO_06, NEO_07, NEO_08, NEO_09, NEO_10, NEO_11, NEO_12: WS2812B_5050N, adafruit:WS2812B_5050N
- removed U$5: DUAL1865_BATTERY_HOLDER_NO_CON, nathans-custom-parts:DUAL1865_BATTERY_HOLDER_NO_CON
- added 5V_TEST, BAT_TEST: (no value), pinhead:PINHD-1X2
- added C6, C8: 0.1uF, adafruit:C-USC1206K
- added C7, C9: 200pF, adafruit:C-USC1206K
- added I2C_SEL: FEMALE 2x3, SparkFun-Connectors:CONN_03X2FEMALE
- added MK_FRONT, MK_REAR: SPH0645LM4H-B, SPH0645LM4H-B:SPH0645LM4H-B
- added NEO1, NEO10, NEO2, NEO3, NEO4, NEO5, NEO6, NEO7, NEO8, NEO9: WS2812B5050, adafruit:WS2812B5050
- added NEOP: B3B-PH-K, con-jst-ph:B3B-PH-K
- added NEOP_T1, NEOP_T2: B2B-PH-K, con-jst-ph:B2B-PH-K
- added R10, R11, R12, R15: 68R, adafruit:R-US_M1206
- added U$2: BK-18650-PC4, BK-18650-PC4:BK-18650-PC4
- added U$3: TEENSY_3.1-3.2_DIL, Teensy_3_and_LC_Series_Boards_v1.4:TEENSY_3.1-3.2_DIL
- C1, C13, C15, C2, C21, C3, C4, NC1, NC10, NC2, NC3, NC4, NC5, NC6, NC7, NC8, NC9: device SparkFun-Capacitors:5.6PF-0603-50V-5% -> adafruit:C-USC1206K
- C14: value 33uf_50v -> 33uf
- MEMS_FRONT, MEMS_REAR: value SPH0645 -> B6B-PH-K; device nathans-custom-parts:SPH0645_MEMS_MICROPHONE -> con-jst-ph:B6B-PH-K
- R1, R2, R5, R6, R7, R8, R9: device adafruit:R-US_0207/10 -> adafruit:R-US_R1206W
- R3, R4: device SparkFun-Resistors:4.7KOHM-0603-1/10W-1% -> adafruit:R-US_R1206W
Connections:
- removed net N$13: NEO_09.DO, NEO_10.DI
- removed net N$14: NEO_10.DO, NEO_11.DI
- new net AGND: C6.2, C7.2, C8.2, C9.2, MEMS_FRONT.2, MEMS_REAR.2, MK_FRONT.GND, MK_REAR.GND, U$3.AGND
- new net BCLK_P: MK_FRONT.BCLK, MK_REAR.BCLK, R11.1
- new net DIN: R12.2, R15.2, U$3.13/SCK/LED
- new net LRCLK_P: MK_FRONT.WS, MK_REAR.WS, R10.1
- new net N$17: MK_REAR.DATA_OUT, R15.1
- new net N$20: U$2.+2, U$2.-1
- new net N$3: MK_FRONT.DATA_OUT, R12.1
- net 3.3V: now also C13.1, C15.1, C6.1, C7.1, C8.1, C9.1, MEMS_FRONT.1, MEMS_FRONT.6, MEMS_REAR.1, MK_FRONT.SELECT, MK_FRONT.VDD, MK_REAR.VDD, U$3.3.3V; no longer 3.3V.P$1, B1.3.3V, C13.2, C15.2, MEMS_FRONT.3V, MEMS_FRONT.SEL, MEMS_REAR.3V
- net 5V: now also 5V_TEST.1, C21.1, NEO1.VDD, NEO10.VDD, NEO2.VDD, NEO3.VDD, NEO4.VDD, NEO5.VDD, NEO6.VDD, NEO7.VDD, NEO8.VDD, NEO9.VDD, NEOP.1, U$3.VIN; no longer 5V.P$1, C21.2, NC11.1, NC12.1, NEO_01.VDD, NEO_02.VDD, NEO_03.VDD, NEO_04.VDD, NEO_05.VDD, NEO_06.VDD, NEO_07.VDD, NEO_08.VDD, NEO_09.VDD, NEO_10.VDD, NEO_11.VDD, NEO_12.VDD
- net BAT_IN: now also BAT_TEST.1, U$2.+1; no longer BAT+.P$1, BAT_IN.1
- net BCLK: now also MEMS_FRONT.3, MEMS_REAR.3, R11.2, U$3.9/RX2/PWM; no longer MEMS_FRONT.BCLK, MEMS_REAR.BCLK
- net GND: now also 5V_TEST.2, BAT_TEST.2, C13.2, C15.2, C21.2, MEMS_REAR.6, MK_REAR.SELECT, NEO1.GND, NEO10.GND, NEO2.GND, NEO3.GND, NEO4.GND, NEO5.GND, NEO6.GND, NEO7.GND, NEO8.GND, NEO9.GND, NEOP.3, NEOP_T1.2, NEOP_T2.2, U$2.-2, U$3.GND; no longer BAT_IN.2, C13.1, C15.1, C21.1, GND.P$1, MEMS_FRONT.GND, MEMS_REAR.GND, MEMS_REAR.SEL, NC11.2, NC12.2, NEO_01.GND, NEO_02.GND, NEO_03.GND, NEO_04.GND, NEO_05.GND, NEO_06.GND, NEO_07.GND, NEO_08.GND, NEO_09.GND, NEO_10.GND, NEO_11.GND, NEO_12.GND
- net I2C_RESET: now also U$3.20/A6/PWM
- net I2S_DATA: now also MEMS_FRONT.4, MEMS_REAR.4; no longer MEMS_FRONT.DOUT, MEMS_REAR.DOUT
- net LRCLK: now also MEMS_FRONT.5, MEMS_REAR.5, R10.2, U$3.23/A9/T/PWM; no longer MEMS_FRONT.LRCL, MEMS_REAR.LRCL
- net N$10: now also NEO3.DO, NEO4.DI; no longer NEO_03.DO, NEO_04.DI
- net N$11: now also NEO7.DO, NEO8.DI; no longer NEO_07.DO, NEO_08.DI
- net N$12: now also NEO8.DO, NEO9.DI; no longer NEO_08.DO, NEO_09.DI
- net N$23: now also NEO6.DO, NEO7.DI; no longer NEO_06.DO, NEO_07.DI
- net N$4: now also NEO2.DO, NEO3.DI; no longer NEO_02.DO, NEO_03.DI
- net N$5: now also NEO5.DO, NEO6.DI, NEOP_T1.1; no longer NEO_05.DO, NEO_06.DI
- net N$6: now also NEO10.DI, NEO9.DO, NEOP_T2.1; no longer NEO_11.DO, NEO_12.DI
- net N$8: now also NEO4.DO, NEO5.DI; no longer NEO_04.DO, NEO_05.DI
- net NEO_P1: now also NEO1.DO, NEO2.DI; no longer NEO_01.DO, NEO_02.DI
- net NEO_P_CTRL: now also NEO1.DI, NEOP.2, U$3.5/PWM; no longer NEO_01.DI
- net SCL: now also I2C_SEL.4, U$3.19/A5/T/SCL0; no longer B1.A5/19/SCL0, SCL.P$1
- net SCL0: now also I2C_SEL.2; no longer SCL0.P$1
- net SCL1: now also I2C_SEL.6; no longer SCL1.P$1
- net SDA: now also I2C_SEL.3, U$3.18/A4/T/SDA0; no longer B1.A4/18/SDA0, SDA.P$1
- net SDA0: now also I2C_SEL.1; no longer SDA0.P$1
- net SDA1: now also I2C_SEL.5; no longer SDA1.P$1
Other:
- note added: "10R"
- note added: "14/10/2019"
- note added: "Designed by Nathan Villicana-Shaw Victoria University of Wellington School of Engineering and Computer Science"
- note added: "R10 and R11 need to be as close as possible to the Teensy"
- note added: "R12 should be close to mic"
- note removed: "Add Test Pads to several of the LEDs"
- note removed: "Change all components to 1206 instead of 0603"
- note removed: "First 6 NeoPixels are on the front of the board while the remaining 6 are "off board""
- note removed: "Keep the I2C jst connectors for test points, but do not populate with parts?"
- note removed: "Make the NeoP footprint have wider/longer pads for soldering to"
- note removed: "Should be larger!!!! Not able to use most/many of these!"
- note removed: "Test Points"
- note removed: "The lux sensor has a fixed I2C address the bus expander allows us to talk to both on the same bus"
- note removed: "Unidirectional buffer chips like 74HCT245 and 74AHCT125 are"
- note removed: "Wow, the pwr switch needs to be connected to the pwr reg dummy!"
- note removed: "replace 10uf cap with 1206"
- moved on the sheet: C13, C14, C15, C21, C5, MEMS_FRONT, MEMS_REAR, NC1, NC10, NC2, NC3, NC4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
