File: PCB/v3/54mm_breakout/moth_v3_54mm_breakout.brd (EAGLE design)
At the start: 55 x 55 mm, 31 parts

Commit message: minor changes to the v3 breakout and main board
Other:
- board text added: "Serial"
- board text added: "Tested"
Changed lines of the file:
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@@
 <grid distance="0.5" unitdist="mil" unit="mil" style="dots" multiple="1" display="yes" altdistance="0.25" altunitdist="mil" altunit="mil"/>
 <layers>
-<layer number="1" name="Top" color="4" fill="1" visible="yes" active="yes"/>
-<layer number="2" name="Route2" color="16" fill="1" visible="yes" active="yes"/>
+<layer number="1" name="Top" color="4" fill="1" visible="no" active="yes"/>
+<layer number="2" name="Route2" color="16" fill="1" visible="no" active="yes"/>
 <layer number="3" name="Route3" color="17" fill="1" visible="no" active="no"/>
 <layer number="4" name="Route4" color="18" fill="1" visible="no" active="no"/>
@@
 <layer number="19" name="Unrouted" color="6" fill="1" visible="yes" active="yes"/>
 <layer number="20" name="Dimension" color="24" fill="1" visible="yes" active="yes"/>
-<layer number="21" name="tPlace" color="7" fill="1" visible="yes" active="yes"/>
+<layer number="21" name="tPlace" color="7" fill="1" visible="no" active="yes"/>
 <layer number="22" name="bPlace" color="7" fill="1" visible="yes" active="yes"/>
-<layer number="23" name="tOrigins" color="15" fill="1" visible="yes" active="yes"/>
+<layer number="23" name="tOrigins" color="15" fill="1" visible="no" active="yes"/>
 <layer number="24" name="bOrigins" color="15" fill="1" visible="yes" active="yes"/>
-<layer number="25" name="tNames" color="7" fill="1" visible="yes" active="yes"/>
+<layer number="25" name="tNames" color="7" fill="1" visible="no" active="yes"/>
 <layer number="26" name="bNames" color="7" fill="1" visible="yes" active="yes"/>
 <layer number="27" name="tValues" color="7" fill="1" visible="no" active="yes"/>
@@
 <layer number="37" name="tTest" color="7" fill="1" visible="no" active="yes"/>
 <layer number="38" name="bTest" color="7" fill="1" visible="no" active="yes"/>
-<layer number="39" name="tKeepout" color="4" fill="11" visible="yes" active="yes"/>
+<layer number="39" name="tKeepout" color="4" fill="11" visible="no" active="yes"/>
 <layer number="40" name="bKeepout" color="1" fill="11" visible="yes" active="yes"/>
-<layer number="41" name="tRestrict" color="4" fill="10" visible="yes" active="yes"/>
+<layer number="41" name="tRestrict" color="4" fill="10" visible="no" active="yes"/>
 <layer number="42" name="bRestrict" color="1" fill="10" visible="yes" active="yes"/>
 <layer number="43" name="vRestrict" color="2" fill="10" visible="no" active="yes"/>
@@
 <layer number="49" name="Reference" color="7" fill="1" visible="no" active="yes"/>
 <layer number="50" name="dxf" color="7" fill="1" visible="no" active="no"/>
-<layer number="51" name="tDocu" color="7" fill="1" visible="yes" active="yes"/>
+<layer number="51" name="tDocu" color="7" fill="1" visible="no" active="yes"/>
 <layer number="52" name="bDocu" color="7" fill="1" visible="yes" active="yes"/>
 <layer number="53" name="tGND_GNDA" color="7" fill="9" visible="no" active="no"/>
@@
 <rectangle x1="0.04445" y1="0.24765" x2="0.05715" y2="0.26035" layer="22"/>
 <text x="-0.7366" y="-4.1783" size="0.8128" layer="22" font="vector" ratio="12" rot="MR0" align="center">200pf</text>
-<text x="-14.1224" y="20.8534" size="0.8128" layer="22" font="vector" ratio="12" rot="MR270" align="top-left">5V
+<text x="-5.3213" y="20.5486" size="1.27" layer="22" font="vector" ratio="12" rot="MR270" align="top-left">5V
 NOUT
 SCL
@@
 POL
 GND</text>
-<text x="-14.097" y="15.1765" size="0.8128" layer="22" font="vector" ratio="12" rot="MR270" align="top-right">3.3V
+<text x="-5.3594" y="11.0744" size="1.27" layer="22" font="vector" ratio="12" rot="MR270" align="top-right">3.3V
 NIN
 SDA
@@
 LRC
 GND</text>
-<wire x1="-14.3637" y1="20.8915" x2="-14.3637" y2="17.7546" width="0.254" layer="22"/>
 <wire x1="-14.3637" y1="17.7546" x2="-14.3637" y2="17.7292" width="0.254" layer="22"/>
-<wire x1="-14.3637" y1="17.7292" x2="-6.9342" y2="17.7292" width="0.254" layer="22"/>
-<wire x1="-6.9342" y1="17.7292" x2="-6.9342" y2="20.9042" width="0.254" layer="22"/>
-<wire x1="-6.9342" y1="20.9042" x2="-13.1445" y2="20.9042" width="0.254" layer="22"/>
-<wire x1="-13.1445" y1="20.9042" x2="-14.3764" y2="20.9042" width="0.254" layer="22"/>
-<wire x1="-6.9469" y1="17.7546" x2="-6.9469" y2="14.6812" width="0.254" layer="22"/>
-<wire x1="-6.9469" y1="14.6812" x2="-14.37005" y2="14.64945" width="0.254" layer="22"/>
-<wire x1="-14.37005" y1="14.64945" x2="-14.37005" y2="17.72285" width="0.254" layer="22"/>
-<wire x1="-14.37005" y1="17.72285" x2="-14.3637" y2="17.7546" width="0.254" layer="22"/>
-<wire x1="-13.1826" y1="14.605" x2="-13.1445" y2="14.605" width="0.1016" layer="22"/>
-<wire x1="-13.1445" y1="14.605" x2="-13.1445" y2="20.9042" width="0.1016" layer="22"/>
-<wire x1="-13.1445" y1="20.9042" x2="-11.9126" y2="20.9042" width="0.1016" layer="22"/>
-<wire x1="-11.9126" y1="20.9042" x2="-11.9126" y2="14.6304" width="0.1016" layer="22"/>
-<wire x1="-11.9126" y1="14.6304" x2="-10.6934" y2="14.6304" width="0.1016" layer="22"/>
-<wire x1="-10.6934" y1="14.6304" x2="-10.6934" y2="20.8788" width="0.1016" layer="22"/>
-<wire x1="-10.6934" y1="20.8788" x2="-9.4869" y2="20.8788" width="0.1016" layer="22"/>
-<wire x1="-9.4869" y1="20.8788" x2="-9.4869" y2="14.6939" width="0.1016" layer="22"/>
-<wire x1="-9.4869" y1="14.6939" x2="-8.1534" y2="14.6939" width="0.1016" layer="22"/>
-<wire x1="-8.1534" y1="14.6939" x2="-8.1534" y2="20.8661" width="0.1016" layer="22"/>
+<text x="-12.2428" y="-6.0579" size="1.778" layer="26" rot="MR270">Serial</text>
+<rectangle x1="-10.9982" y1="-12.6365" x2="-0.9144" y2="-6.0579" layer="26"/>
+<text x="2.2733" y="-6.0579" size="1.778" layer="26" rot="MR270">Tested</text>
+<rectangle x1="3.2512" y1="-12.5095" x2="12.954" y2="-6.1849" layer="26"/>
+<wire x1="-5.8293" y1="15.6845" x2="-5.8293" y2="10.5791" width="0.4064" layer="26"/>
+<wire x1="-5.8293" y1="10.5791" x2="5.9182" y2="10.4902" width="0.4064" layer="26"/>
+<wire x1="5.9182" y1="10.4902" x2="5.9182" y2="15.5956" width="0.4064" layer="26"/>
+<wire x1="5.9182" y1="15.5956" x2="6.0198" y2="20.8026" width="0.4064" layer="26"/>
+<wire x1="6.0198" y1="20.8026" x2="-5.7912" y2="20.8026" width="0.4064" layer="26"/>
+<wire x1="-5.7912" y1="20.8026" x2="-5.7912" y2="15.6845" width="0.4064" layer="26"/>
+<wire x1="-5.7912" y1="15.6845" x2="5.9182" y2="15.5956" width="0.4064" layer="26"/>
 </plain>
 <attributes>
@@
 <attribute name="POPULARITY" value="63" x="5.4861" y="7.2091" size="1.778" layer="27" display="off"/>
 <attribute name="SPICEPREFIX" value="C" x="5.4861" y="7.2091" size="1.778" layer="27" display="off"/>
-<attribute name="VALUE" x="7.06155" y="9.17545" size="0.8128" layer="25" ratio="12" rot="R180"/>
+<attribute name="VALUE" x="10.47785" y="7.66415" size="0.8128" layer="25" ratio="12" rot="R180"/>
 </element>
 <element name="C2" library="rcl" library_urn="urn:adsk.eagle:library:334" package="C0805" package3d_urn="urn:adsk.eagle:package:23617/2" value="10uf" x="5.4756" y="5.0984" smashed="yes">
 <attribute name="POPULARITY" value="63" x="5.4756" y="5.0984" size="1.778" layer="27" display="off"/>
 <attribute name="SPICEPREFIX" value="C" x="5.4756" y="5.0984" size="1.778" layer="27" display="off"/>
-<attribute name="VALUE" x="7.61375" y="5.59005" size="0.8128" layer="25" ratio="12"/>
+<attribute name="VALUE" x="7.82965" y="4.81535" size="0.8128" layer="25" ratio="12"/>
 </element>
 <element name="R2" library="adafruit" library_urn="urn:adsk.eagle:library:420" package="M0805" package3d_urn="urn:adsk.eagle:package:6240587/1" value="68R" x="5.055" y="-0.0169" smashed="yes" rot="MR180">
@@
 <attribute name="SPICEPREFIX" value="C" x="-9.0678" y="-44.3968" size="1.778" layer="27" display="off"/>
 </element>
-<element name="INPUT" library="nathans-custom-parts" package="SAMTEC_ESQT_2X6_THROUGH_HOLE" override_package3d_urn="urn:adsk.eagle:package:19145965/2" override_package_urn="urn:adsk.eagle:footprint:19145966/1" value="ESQT" x="0" y="22.75" locked="yes" smashed="yes" rot="MR0">
-<attribute name="NAME" x="-0.25" y="19.545" locked="yes" size="2" layer="26" font="vector" ratio="12" rot="MR180" align="center"/>
+<element name="INPUT" library="nathans-custom-parts" package="SAMTEC_ESQT_2X6_THROUGH_HOLE" override_package3d_urn="urn:adsk.eagle:package:19145965/2" override_package_urn="urn:adsk.eagle:footprint:19145966/1" value="ESQT" x="0" y="22.75" smashed="yes" rot="MR0">
+<attribute name="NAME" x="7.4171" y="22.5084" size="1.778" layer="26" font="vector" ratio="12" rot="MR90" align="center"/>
 </element>
 <element name="OUTPUT" library="nathans-custom-parts" library_urn="urn:adsk.eagle:library:19144427" package="SAMTEC_TW_2X6" package3d_urn="urn:adsk.eagle:package:19144521/1" override_package3d_urn="urn:adsk.eagle:package:19146336/2" override_package_urn="urn:adsk.eagle:footprint:19146337/1" override_locally_modified="yes" value="TW" x="0" y="-22.75" locked="yes" smashed="yes" rot="MR0">
